File: 24Vin.sch (KiCad schematic (older format))
At the start: 26 parts

Commit message: Added all stepper circuits. Adding SPI bus to top level sheet. Opened up layout to check connectivity. Errors with footprint libs
Parts:
- gave numbers to parts that had none: 26

Commit message: added RESET and XTAL to atmega2560
Parts:
- added SW301: SW_Push, symbol Switch:SW_Push
- added TP301: TestPoint, symbol Connector:TestPoint
- C1: value C -> 0.01uF
Connections:
- net +5V: now also TP301.1
- net GND: now also SW301.1
- net at R3.2, R5.1, TP1.1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: now also SW301.2
Other:
- note added: "Needs to be XXX 430.\n431 is about5-23V...\nVin = 24V\n"
- note added: "Pulling EN low resets TPS"
- note added: "need low ESR, X7R or X5R"
- moved on the sheet: C2, C3, L1
Changed lines of the file:
@@
 	3800 1400 3800 1300
 Wire Wire Line
-	3800 1500 3800 1400
+	3800 1500 3800 1450
 Connection ~ 3800 1400
 $Comp
@@
 	1300 1100 1300 1350
 Wire Wire Line
-	3800 1800 3800 2050
+	3800 1800 3800 1900
 $Comp
 L power:GND #PWR0103
@@
 P 5900 1000
 F 0 "C1" V 5648 1000 50  0000 C CNN
-F 1 "C" V 5739 1000 50  0000 C CNN
+F 1 "0.01uF" V 5739 1000 50  0000 C CNN
 F 2 "" H 5938 850 50  0001 C CNN
 F 3 "~" H 5900 1000 50  0001 C CNN
@@
 L Device:L L1
 U 1 1 5EE87364
-P 2850 1000
-F 0 "L1" V 2669 1000 50  0000 C CNN
-F 1 "L" V 2760 1000 50  0000 C CNN
-F 2 "" H 2850 1000 50  0001 C CNN
-F 3 "~" H 2850 1000 50  0001 C CNN
-	1    2850 1000
+P 2500 1000
+F 0 "L1" V 2319 1000 50  0000 C CNN
+F 1 "L" V 2410 1000 50  0000 C CNN
+F 2 "" H 2500 1000 50  0001 C CNN
+F 3 "~" H 2500 1000 50  0001 C CNN
+	1    2500 1000
 	0    1    1    0
 $EndComp
 Wire Wire Line
-	2250 1000 2700 1000
-Wire Wire Line
-	3000 1000 3200 1000
+	2250 1000 2350 1000
+Wire Wire Line
+	2650 1000 2800 1000
 Connection ~ 3800 1000
 $Comp
 L Device:C C2
 U 1 1 5EE88BE8
-P 3200 1150
-F 0 "C2" H 3315 1196 50  0000 L CNN
-F 1 "C" H 3315 1105 50  0000 L CNN
-F 2 "" H 3238 1000 50  0001 C CNN
-F 3 "~" H 3200 1150 50  0001 C CNN
-	1    3200 1150
-	1    0    0    -1
-$EndComp
-Connection ~ 3200 1000
-Wire Wire Line
-	3200 1000 3550 1000
+P 2800 1150
+F 0 "C2" H 2915 1196 50  0000 L CNN
+F 1 "C" H 2915 1105 50  0000 L CNN
+F 2 "" H 2838 1000 50  0001 C CNN
+F 3 "~" H 2800 1150 50  0001 C CNN
+	1    2800 1150
+	1    0    0    -1
+$EndComp
 $Comp
 L Device:C C3
 U 1 1 5EE88FF0
-P 3550 1150
-F 0 "C3" H 3665 1196 50  0000 L CNN
-F 1 "C" H 3665 1105 50  0000 L CNN
-F 2 "" H 3588 1000 50  0001 C CNN
-F 3 "~" H 3550 1150 50  0001 C CNN
-	1    3550 1150
-	1    0    0    -1
-$EndComp
-Connection ~ 3550 1000
-Wire Wire Line
-	3550 1000 3800 1000
+P 3150 1150
+F 0 "C3" H 3265 1196 50  0000 L CNN
+F 1 "C" H 3265 1105 50  0000 L CNN
+F 2 "" H 3188 1000 50  0001 C CNN
+F 3 "~" H 3150 1150 50  0001 C CNN
+	1    3150 1150
+	1    0    0    -1
+$EndComp
 $Comp
 L power:GND #PWR0104
 U 1 1 5EE89390
-P 3350 1350
-F 0 "#PWR0104" H 3350 1100 50  0001 C CNN
-F 1 "GND" H 3355 1177 50  0000 C CNN
-F 2 "" H 3350 1350 50  0001 C CNN
-F 3 "" H 3350 1350 50  0001 C CNN
-	1    3350 1350
-	1    0    0    -1
-$EndComp
-Wire Wire Line
-	3200 1300 3200 1350
-Wire Wire Line
-	3200 1350 3350 1350
-Wire Wire Line
-	3550 1350 3550 1300
-Connection ~ 3350 1350
-Wire Wire Line
-	3350 1350 3550 1350
+P 2950 1400
+F 0 "#PWR0104" H 2950 1150 50  0001 C CNN
+F 1 "GND" H 2955 1227 50  0000 C CNN
+F 2 "" H 2950 1400 50  0001 C CNN
+F 3 "" H 2950 1400 50  0001 C CNN
+	1    2950 1400
+	1    0    0    -1
+$EndComp
 $Comp
 L Device:D_Schottky D1
@@
 Connection ~ 7850 1800
 Wire Wire Line
-	7850 1000 7200 1000
+	7850 1000 7450 1000
 Connection ~ 7200 1000
 $Comp
@@
 Wire Wire Line
 	4050 1400 3800 1400
+$Comp
+L Connector:TestPoint TP301
+U 1 1 619B2B76
+P 7450 1000
+F 0 "TP301" H 7508 1118 50  0000 L CNN
+F 1 "TestPoint" H 7508 1027 50  0000 L CNN
+F 2 "" H 7650 1000 50  0001 C CNN
+F 3 "~" H 7650 1000 50  0001 C CNN
+	1    7450 1000
+	1    0    0    -1
+$EndComp
+Connection ~ 7450 1000
+Wire Wire Line
+	7450 1000 7200 1000
+Connection ~ 2800 1000
+Wire Wire Line
+	2800 1000 3150 1000
+Connection ~ 3150 1000
+Wire Wire Line
+	3150 1000 3800 1000
+Wire Wire Line
+	2800 1300 2800 1350
+Wire Wire Line
+	2800 1350 2950 1350
+Wire Wire Line
+	3150 1350 3150 1300
+Wire Wire Line
+	2950 1350 2950 1400
+Connection ~ 2950 1350
+Wire Wire Line
+	2950 1350 3150 1350
+$Comp
+L Switch:SW_Push SW301
+U 1 1 619BC547
+P 3350 1700
+F 0 "SW301" V 3396 1652 50  0000 R CNN
+F 1 "SW_Push" V 3305 1652 50  0000 R CNN
+F 2 "" H 3350 1900 50  0001 C CNN
+F 3 "" H 3350 1900 50  0001 C CNN
+	1    3350 1700
+	0    -1   -1   0
+$EndComp
+Wire Wire Line
+	3800 1450 3350 1450
+Wire Wire Line
+	3350 1450 3350 1500
+Connection ~ 3800 1450
+Wire Wire Line
+	3800 1450 3800 1400
+Wire Wire Line
+	3350 1900 3800 1900
+Connection ~ 3800 1900
+Wire Wire Line
+	3800 1900 3800 2050
+Text Notes 2400 2150 0    59   ~ 0
+Pulling EN low resets TPS
+Wire Notes Line
+	3400 1400 3400 2000
+Wire Notes Line
+	3400 2000 3150 2000
+Wire Notes Line
+	3150 2000 3150 1400
+Wire Notes Line
+	3150 1400 3400 1400
+Text Notes 5350 700  0    59   ~ 0
+need low ESR, X7R or X5R
+Text Notes 4200 750  0    59   ~ 0
+Needs to be XXX 430.\n431 is about5-23V...\nVin = 24V\n
 $EndSCHEMATC

Commit message: updated ATMEGA and regulators
Parts:
- removed R3, R5: R, symbol Device:R
- removed SW301: SW_Push, symbol Switch:SW_Push
- removed TP1: TestPoint, symbol Connector:TestPoint
- removed U3: TPS5431DDA, Package_SO:TI_SO-PowerPAD-8_ThermalVias, symbol Regulator_Switching:TPS5431DDA
- added D? (x2): LED, symbol Device:LED
- added R? (x2): R, symbol Device:R
- added TP? (x2): TestPoint, symbol Connector:TestPoint
- added U3: TPS5430DDA, Package_SO:TI_SO-PowerPAD-8_ThermalVias, symbol Regulator_Switching:TPS5430DDA
- C3: value C -> 10uF
- C4: value CP1 -> 220uF
- L2: value L -> 15uH
- R4: value R -> 10k
- R6: value R -> 3.34k
Connections:
- net +3V3: now also D?.2 (A)
- net +5V: now also D?.2 (A)
- net GND: now also R?.2, R?.2, TP?.1, U3.6 (GND), U3.9 (GNDPAD)
- net at C1.2: now also U3.1 (BOOT)
- net at R4.2, R6.1: now also U3.4 (VSENSE)
- net at C2.1, C3.1, L1.1: now also U3.7 (VIN)
- net at C1.1, D1.1 (K), L2.2: now also U3.8 (PH)
- new net: D?.1 (K), R?.1 (x2)
- new net: TP?.1, U3.5 (EN)
Other:
- note added: "Pulling EN low resets TPS\nInternal Pullup\n"
- note removed: "Needs to be XXX 430.\n431 is about5-23V...\nVin = 24V\n"
- note removed: "Pulling EN low resets TPS"
- moved on the sheet: R4, R6, TP301
Changed lines of the file:
@@
 	0    1    1    0
 $EndComp
-$Comp
-L Regulator_Switching:TPS5431DDA U3
-U 1 1 5EE7FA31
-P 4900 1200
-F 0 "U3" H 4900 1667 50  0000 C CNN
-F 1 "TPS5431DDA" H 4900 1576 50  0000 C CNN
-F 2 "Package_SO:TI_SO-PowerPAD-8_ThermalVias" H 4950 850 50  0001 L CIN
-F 3 "http://www.ti.com/lit/ds/symlink/tps5430.pdf" H 4900 1200 50  0001 C CNN
-	1    4900 1200
-	1    0    0    -1
-$EndComp
-Wire Wire Line
-	4400 1000 3800 1000
 Wire Wire Line
 	1950 1000 1100 1000
-$Comp
-L Device:R R3
-U 1 1 5EE838EE
-P 3800 1150
-F 0 "R3" H 3870 1196 50  0000 L CNN
-F 1 "R" H 3870 1105 50  0000 L CNN
-F 2 "" V 3730 1150 50  0001 C CNN
-F 3 "~" H 3800 1150 50  0001 C CNN
-	1    3800 1150
-	1    0    0    -1
-$EndComp
-$Comp
-L Device:R R5
-U 1 1 5EE83BF6
-P 3800 1650
-F 0 "R5" H 3870 1696 50  0000 L CNN
-F 1 "R" H 3870 1605 50  0000 L CNN
-F 2 "" V 3730 1650 50  0001 C CNN
-F 3 "~" H 3800 1650 50  0001 C CNN
-	1    3800 1650
-	1    0    0    -1
-$EndComp
 Wire Wire Line
 	4400 1400 4050 1400
-Wire Wire Line
-	3800 1400 3800 1300
-Wire Wire Line
-	3800 1500 3800 1450
-Connection ~ 3800 1400
 $Comp
 L power:GND #PWR0101
@@
 L power:GND #PWR0102
 U 1 1 5EE848A6
-P 3800 2050
-F 0 "#PWR0102" H 3800 1800 50  0001 C CNN
-F 1 "GND" H 3805 1877 50  0000 C CNN
-F 2 "" H 3800 2050 50  0001 C CNN
-F 3 "" H 3800 2050 50  0001 C CNN
-	1    3800 2050
+P 3800 1850
+F 0 "#PWR0102" H 3800 1600 50  0001 C CNN
+F 1 "GND" H 3805 1677 50  0000 C CNN
+F 2 "" H 3800 1850 50  0001 C CNN
+F 3 "" H 3800 1850 50  0001 C CNN
+	1    3800 1850
 	1    0    0    -1
 $EndComp
@@
 Wire Wire Line
 	1300 1100 1300 1350
-Wire Wire Line
-	3800 1800 3800 1900
 $Comp
 L power:GND #PWR0103
@@
 P 6750 1000
 F 0 "L2" V 6569 1000 50  0000 C CNN
-F 1 "L" V 6660 1000 50  0000 C CNN
+F 1 "15uH" V 6660 1000 50  0000 C CNN
 F 2 "" H 6750 1000 50  0001 C CNN
 F 3 "~" H 6750 1000 50  0001 C CNN
@@
 Wire Wire Line
 	2650 1000 2800 1000
-Connection ~ 3800 1000
 $Comp
 L Device:C C2
@@
 P 3150 1150
 F 0 "C3" H 3265 1196 50  0000 L CNN
-F 1 "C" H 3265 1105 50  0000 L CNN
+F 1 "10uF" H 3265 1105 50  0000 L CNN
 F 2 "" H 3188 1000 50  0001 C CNN
 F 3 "~" H 3150 1150 50  0001 C CNN
@@
 P 7200 1250
 F 0 "C4" H 7315 1296 50  0000 L CNN
-F 1 "CP1" H 7315 1205 50  0000 L CNN
+F 1 "220uF" H 7315 1205 50  0000 L CNN
 F 2 "" H 7200 1250 50  0001 C CNN
 F 3 "~" H 7200 1250 50  0001 C CNN
@@
 L Device:R R4
 U 1 1 5EE93935
-P 7850 1150
-F 0 "R4" H 7920 1196 50  0000 L CNN
-F 1 "R" H 7920 1105 50  0000 L CNN
-F 2 "" V 7780 1150 50  0001 C CNN
-F 3 "~" H 7850 1150 50  0001 C CNN
-	1    7850 1150
+P 7800 1450
+F 0 "R4" H 7870 1496 50  0000 L CNN
+F 1 "10k" H 7870 1405 50  0000 L CNN
+F 2 "" V 7730 1450 50  0001 C CNN
+F 3 "~" H 7800 1450 50  0001 C CNN
+	1    7800 1450
 	1    0    0    -1
 $EndComp
@@
 L Device:R R6
 U 1 1 5EE94277
-P 7850 1950
-F 0 "R6" H 7920 1996 50  0000 L CNN
-F 1 "R" H 7920 1905 50  0000 L CNN
-F 2 "" V 7780 1950 50  0001 C CNN
-F 3 "~" H 7850 1950 50  0001 C CNN
-	1    7850 1950
+P 7800 1950
+F 0 "R6" H 7870 1996 50  0000 L CNN
+F 1 "3.34k" H 7870 1905 50  0000 L CNN
+F 2 "" V 7730 1950 50  0001 C CNN
+F 3 "~" H 7800 1950 50  0001 C CNN
+	1    7800 1950
 	1    0    0    -1
 $EndComp
@@
 Wire Wire Line
 	5550 1400 5550 1800
-Wire Wire Line
-	5550 1800 7850 1800
-Wire Wire Line
-	7850 1300 7850 1800
-Connection ~ 7850 1800
-Wire Wire Line
-	7850 1000 7450 1000
 Connection ~ 7200 1000
 $Comp
@@
 	1    0    0    -1
 $EndComp
-Wire Wire Line
-	7850 2200 7850 2100
 $Comp
 L power:+5V #PWR0108
@@
 $EndComp
 Wire Wire Line
-	8050 1000 7850 1000
-Wire Wire Line
 	8050 850  8050 1000
-Connection ~ 7850 1000
 $Comp
 L Regulator_Linear:AMS1117-3.3 U4
@@
 	2350 3300 2400 3300
 Wire Wire Line
-	3000 3300 3000 3100
+	3000 3300 3000 3200
 $Comp
 L Device:C C6
@@
 Wire Wire Line
 	2750 5600 2900 5600
-$Comp
-L Connector:TestPoint TP1
-U 1 1 5EEE2BF1
+Wire Wire Line
+	4050 1250 4050 1400
+Connection ~ 7450 1000
+Wire Wire Line
+	7450 1000 7200 1000
+Connection ~ 2800 1000
+Wire Wire Line
+	2800 1000 3150 1000
+Connection ~ 3150 1000
+Wire Wire Line
+	2800 1300 2800 1350
+Wire Wire Line
+	2800 1350 2950 1350
+Wire Wire Line
+	3150 1350 3150 1300
+Wire Wire Line
+	2950 1350 2950 1400
+Connection ~ 2950 1350
+Wire Wire Line
+	2950 1350 3150 1350
+Text Notes 5350 700  0    59   ~ 0
+need low ESR, X7R or X5R
+$Comp
+L Device:LED D?
+U 1 1 62235D6D
+P 8150 1350
+F 0 "D?" V 8189 1232 50  0000 R CNN
+F 1 "LED" V 8098 1232 50  0000 R CNN
+F 2 "" H 8150 1350 50  0001 C CNN
+F 3 "~" H 8150 1350 50  0001 C CNN
+	1    8150 1350
+	0    -1   -1   0
+$EndComp
+$Comp
+L Device:R R?
+U 1 1 62236DFE
+P 8150 1950
+F 0 "R?" H 8220 1996 50  0000 L CNN
+F 1 "R" H 8220 1905 50  0000 L CNN
+F 2 "" V 8080 1950 50  0001 C CNN
+F 3 "~" H 8150 1950 50  0001 C CNN
+	1    8150 1950
+	1    0    0    -1
+$EndComp
+Wire Wire Line
+	8150 1200 8150 1000
+Wire Wire Line
+	8150 1000 8050 1000
+Connection ~ 8050 1000
+Wire Wire Line
+	8150 1500 8150 1800
+Wire Wire Line
+	8150 2100 8150 2150
+$Comp
+L Device:LED D?
+U 1 1 62241ADC
+P 3600 3450
+F 0 "D?" V 3639 3332 50  0000 R CNN
+F 1 "LED" V 3548 3332 50  0000 R CNN
+F 2 "" H 3600 3450 50  0001 C CNN
+F 3 "~" H 3600 3450 50  0001 C CNN
+	1    3600 3450
+	0    -1   -1   0
+$EndComp
+$Comp
+L Device:R R?
+U 1 1 62241AE2
+P 3600 3850
+F 0 "R?" H 3670 3896 50  0000 L CNN
+F 1 "R" H 3670 3805 50  0000 L CNN
+F 2 "" V 3530 3850 50  0001 C CNN
+F 3 "~" H 3600 3850 50  0001 C CNN
+	1    3600 3850
+	1    0    0    -1
+$EndComp
+Wire Wire Line
+	3600 3600 3600 3700
+Wire Wire Line
+	3600 3300 3100 3300
+Connection ~ 3100 3300
+$Comp
+L power:GND #PWR?
+U 1 1 622485D3
+P 3600 4150
+F 0 "#PWR?" H 3600 3900 50  0001 C CNN
+F 1 "GND" H 3605 3977 50  0000 C CNN
+F 2 "" H 3600 4150 50  0001 C CNN
+F 3 "" H 3600 4150 50  0001 C CNN
+	1    3600 4150
+	1    0    0    -1
+$EndComp
+Wire Wire Line
+	3600 4000 3600 4150
+$Comp
+L Regulator_Switching:TPS5430DDA U3
+U 1 1 6224D3F6
+P 4900 1200
+F 0 "U3" H 4900 1667 50  0000 C CNN
+F 1 "TPS5430DDA" H 4900 1576 50  0000 C CNN
+F 2 "Package_SO:TI_SO-PowerPAD-8_ThermalVias" H 4950 850 50  0001 L CIN
+F 3 "http://www.ti.com/lit/ds/symlink/tps5430.pdf" H 4900 1200 50  0001 C CNN
+	1    4900 1200
+	1    0    0    -1
+$EndComp
+Wire Wire Line
+	7800 1000 7800 1300
+Wire Wire Line
+	7800 1600 7800 1800
+Connection ~ 7800 1800
+Wire Wire Line
+	5550 1800 7800 1800
+Connection ~ 7800 1000
+Wire Wire Line
+	7800 1000 7450 1000
+Wire Wire Line
+	7800 1000 8050 1000
+Wire Wire Line
+	7800 2150 7800 2100
+Wire Wire Line
+	7800 2150 7850 2150
+Wire Wire Line
+	7850 2200 7850 2150
+Connection ~ 7850 2150
+Wire Wire Line
+	7850 2150 8150 2150
+Wire Wire Line
+	7450 900  7450 1000
+$Comp
+L Connector:TestPoint TP301
+U 1 1 619B2B76
+P 7450 900
+F 0 "TP301" H 7508 1018 50  0000 L CNN
+F 1 "TestPoint" H 7508 927 50  0000 L CNN
+F 2 "" H 7650 900 50  0001 C CNN
+F 3 "~" H 7650 900 50  0001 C CNN
+	1    7450 900
+	1    0    0    -1
+$EndComp
+Wire Wire Line
+	3150 1000 4400 1000
+Text Notes 3250 1700 0    59   ~ 0
+Pulling EN low resets TPS\nInternal Pullup\n
+$Comp
+L Connector:TestPoint TP?
+U 1 1 62264C9C
+P 3800 1250
+F 0 "TP?" H 3858 1368 50  0000 L CNN
+F 1 "TestPoint" H 3858 1277 50  0001 L CNN
+F 2 "" H 4000 1250 50  0001 C CNN
+F 3 "~" H 4000 1250 50  0001 C CNN
+	1    3800 1250
+	1    0    0    -1
+$EndComp
+$Comp
+L Connector:TestPoint TP?
+U 1 1 62265545
 P 4050 1250
-F 0 "TP1" H 4108 1368 50  0000 L CNN
-F 1 "TestPoint" H 4108 1277 50  0000 L CNN
+F 0 "TP?" H 4108 1368 50  0000 L CNN
+F 1 "TestPoint" H 4108 1277 50  0001 L CNN
 F 2 "" H 4250 1250 50  0001 C CNN
 F 3 "~" H 4250 1250 50  0001 C CNN
@@
 $EndComp
 Wire Wire Line
-	4050 1250 4050 1400
-Connection ~ 4050 1400
-Wire Wire Line
-	4050 1400 3800 1400
-$Comp
-L Connector:TestPoint TP301
-U 1 1 619B2B76
-P 7450 1000
-F 0 "TP301" H 7508 1118 50  0000 L CNN
-F 1 "TestPoint" H 7508 1027 50  0000 L CNN
-F 2 "" H 7650 1000 50  0001 C CNN
-F 3 "~" H 7650 1000 50  0001 C CNN
-	1    7450 1000
-	1    0    0    -1
-$EndComp
-Connection ~ 7450 1000
-Wire Wire Line
-	7450 1000 7200 1000
-Connection ~ 2800 1000
-Wire Wire Line
-	2800 1000 3150 1000
-Connection ~ 3150 1000
-Wire Wire Line
-	3150 1000 3800 1000
-Wire Wire Line
-	2800 1300 2800 1350
-Wire Wire Line
-	2800 1350 2950 1350
-Wire Wire Line
-	3150 1350 3150 1300
-Wire Wire Line
-	2950 1350 2950 1400
-Connection ~ 2950 1350
-Wire Wire Line
-	2950 1350 3150 1350
-$Comp
-L Switch:SW_Push SW301
-U 1 1 619BC547
-P 3350 1700
-F 0 "SW301" V 3396 1652 50  0000 R CNN
-F 1 "SW_Push" V 3305 1652 50  0000 R CNN
-F 2 "" H 3350 1900 50  0001 C CNN
-F 3 "" H 3350 1900 50  0001 C CNN
-	1    3350 1700
-	0    -1   -1   0
-$EndComp
-Wire Wire Line
-	3800 1450 3350 1450
-Wire Wire Line
-	3350 1450 3350 1500
-Connection ~ 3800 1450
-Wire Wire Line
-	3800 1450 3800 1400
-Wire Wire Line
-	3350 1900 3800 1900
-Connection ~ 3800 1900
-Wire Wire Line
-	3800 1900 3800 2050
-Text Notes 2400 2150 0    59   ~ 0
-Pulling EN low resets TPS
-Wire Notes Line
-	3400 1400 3400 2000
-Wire Notes Line
-	3400 2000 3150 2000
-Wire Notes Line
-	3150 2000 3150 1400
-Wire Notes Line
-	3150 1400 3400 1400
-Text Notes 5350 700  0    59   ~ 0
-need low ESR, X7R or X5R
-Text Notes 4200 750  0    59   ~ 0
-Needs to be XXX 430.\n431 is about5-23V...\nVin = 24V\n
+	3800 1250 3800 1850
+$Comp
+L power:VCC #PWR?
+U 1 1 6226C3B6
+P 3350 3100
+F 0 "#PWR?" H 3350 2950 50  0001 C CNN
+F 1 "VCC" H 3365 3273 50  0000 C CNN
+F 2 "" H 3350 3100 50  0001 C CNN
+F 3 "" H 3350 3100 50  0001 C CNN
+	1    3350 3100
+	1    0    0    -1
+$EndComp
+Wire Wire Line
+	3350 3100 3350 3200
+Wire Wire Line
+	3350 3200 3000 3200
+Connection ~ 3000 3200
+Wire Wire Line
+	3000 3200 3000 3100
 $EndSCHEMATC

Commit message: changed ATMEGA vcc to 5V
Changed lines of the file:
@@
 Wire Wire Line
 	2350 3300 2400 3300
-Wire Wire Line
-	3000 3300 3000 3200
 $Comp
 L Device:C C6
@@
 L power:VCC #PWR?
 U 1 1 6226C3B6
-P 3350 3100
-F 0 "#PWR?" H 3350 2950 50  0001 C CNN
-F 1 "VCC" H 3365 3273 50  0000 C CNN
-F 2 "" H 3350 3100 50  0001 C CNN
-F 3 "" H 3350 3100 50  0001 C CNN
-	1    3350 3100
-	1    0    0    -1
-$EndComp
-Wire Wire Line
-	3350 3100 3350 3200
-Wire Wire Line
-	3350 3200 3000 3200
-Connection ~ 3000 3200
-Wire Wire Line
-	3000 3200 3000 3100
+P 8350 850
+F 0 "#PWR?" H 8350 700 50  0001 C CNN
+F 1 "VCC" H 8365 1023 50  0000 C CNN
+F 2 "" H 8350 850 50  0001 C CNN
+F 3 "" H 8350 850 50  0001 C CNN
+	1    8350 850
+	1    0    0    -1
+$EndComp
+Wire Wire Line
+	3000 3100 3000 3300
+Wire Wire Line
+	8150 1000 8350 1000
+Wire Wire Line
+	8350 1000 8350 850
+Connection ~ 8150 1000
 $EndSCHEMATC
