File: FET_drivers.sch (KiCad schematic (older format))
At the start: 62 parts, among them J2 Conn_01x02, J3 Conn_01x02, J4 Conn_01x02, J5 Conn_01x02, Q1 Q_NMOS_GDSD, Q2 Q_NMOS_GDSD, Q3 Q_NMOS_GDSD, Q4 Q_NMOS_GDSD, U5 LM324A

Commit message: added peripherals
Parts:
- removed R20, R21, R22: .02, Resistors_SMD:R_0603_HandSoldering, symbol Device:R
- removed R24, R25, R29, R30, R31, R35, R37: 1k, Resistors_SMD:R_0603_HandSoldering, symbol Device:R
- added R401, R402, R403: .05, Resistors_SMD:R_0603_HandSoldering, symbol Device:R
- added R404, R405, R406, R407, R408, R409, R410: 2k, Resistors_SMD:R_0603_HandSoldering, symbol Device:R
- R19: value .02 -> .05; Manufacturer P/N WSLP1206R0200FEA -> WSLP0805R0500FEB; Vendor P/N WSLP-.02CT-ND -> WSLPB-.05CT-ND
- R23: value 1k -> 2k; Manufacturer P/N CR0603AFX-1001ELF -> CR0603-JW-202ELF; Vendor P/N 118-CR0603AFX-1001ELFCT-ND -> 118-CR0603-JW-202ELFCT-ND
Connections:
- net GND: now also R401.2, R402.2, R403.2, R406.2, R407.2, R408.2, R410.2
- net PERIPH_3: now also R16.2
- net P_1_SENSE: now also R404.2
- net P_2_SENSE: now also R405.2
- net P_3_SENSE: now also R409.2
- net at R32.2, U5.2 (-): now also R406.1
- net at C24.1, U5.5 (+): now also R409.1
- net at R38.2, U5.6 (-): now also R410.1
- net at C19.1, U5.10 (+): now also R404.1
- net at R33.2, U5.9 (-): now also R407.1
- net at C20.1, U5.12 (+): now also R405.1
- net at R34.2, U5.13 (-): now also R408.1
- net at Q2.3 (S): now also R401.1
- net at Q3.3 (S): now also R402.1
- net at Q4.3 (S): now also R403.1
Other:
- note added: "24V Vac Pump\napprox 1A @ 24V\n"
- note removed: "24V Vac Pump\napprox 500mA @ 24V\n"

Commit message: added RESET and XTAL to atmega2560
Parts:
- U5: footprint (none) -> Housings_SOIC:SOIC-14_3.9x8.7mm_Pitch1.27mm
Changed lines of the file:
@@
 F 0 "U5" H 2050 5517 50  0000 C CNN
 F 1 "LM324A" H 2050 5426 50  0000 C CNN
-F 2 "" H 2000 5250 50  0001 C CNN
+F 2 "Housings_SOIC:SOIC-14_3.9x8.7mm_Pitch1.27mm" H 2000 5250 50  0001 C CNN
 F 3 "http://www.ti.com/lit/ds/symlink/lm2902-n.pdf" H 2100 5350 50  0001 C CNN
 	1    2050 5150

Commit message: added footprints for most of the c,r, and tp's. need new buck
Parts:
- U5: footprint (none) -> Housings_SOIC:SOIC-14_3.9x8.7mm_Pitch1.27mm
Changed lines of the file:
@@
 EESchema Schematic File Version 4
-EELAYER 30 0
+LIBS:bountifulHarvest-cache
+EELAYER 26 0
 EELAYER END
 $Descr A4 11693 8268
@@
 F 0 "U5" H 2100 6867 50  0000 C CNN
 F 1 "LM324A" H 2100 6776 50  0000 C CNN
-F 2 "" H 2050 6600 50  0001 C CNN
+F 2 "Housings_SOIC:SOIC-14_3.9x8.7mm_Pitch1.27mm" H 2050 6600 50  0001 C CNN
 F 3 "http://www.ti.com/lit/ds/symlink/lm2902-n.pdf" H 2150 6700 50  0001 C CNN
 	2    2100 6500
@@
 F 0 "U5" H 4900 5617 50  0000 C CNN
 F 1 "LM324A" H 4900 5526 50  0000 C CNN
-F 2 "" H 4850 5350 50  0001 C CNN
+F 2 "Housings_SOIC:SOIC-14_3.9x8.7mm_Pitch1.27mm" H 4850 5350 50  0001 C CNN
 F 3 "http://www.ti.com/lit/ds/symlink/lm2902-n.pdf" H 4950 5450 50  0001 C CNN
 	3    4900 5250
@@
 F 0 "U5" H 8450 5617 50  0000 C CNN
 F 1 "LM324A" H 8450 5526 50  0000 C CNN
-F 2 "" H 8400 5350 50  0001 C CNN
+F 2 "Housings_SOIC:SOIC-14_3.9x8.7mm_Pitch1.27mm" H 8400 5350 50  0001 C CNN
 F 3 "http://www.ti.com/lit/ds/symlink/lm2902-n.pdf" H 8500 5450 50  0001 C CNN
 	4    8450 5250
@@
 F 0 "U5" H 4558 6796 50  0000 L CNN
 F 1 "LM324A" H 4558 6705 50  0000 L CNN
-F 2 "" H 4550 6850 50  0001 C CNN
+F 2 "Housings_SOIC:SOIC-14_3.9x8.7mm_Pitch1.27mm" H 4550 6850 50  0001 C CNN
 F 3 "http://www.ti.com/lit/ds/symlink/lm2902-n.pdf" H 4650 6950 50  0001 C CNN
 	5    4600 6750
