File: STM32.sch (KiCad schematic (older format))
At the start: 21 parts, among them J16 Conn_01x04_Female, U2 STM32F303CBTx

Commit message: added footprints for most of the c,r, and tp's. need new buck
Parts:
- R3, R5: footprint Resistor_SMD:R_0805_2012Metric_Pad1.15x1.40mm_HandSolder -> Resistors_SMD:R_0603_HandSoldering
- U201: renamed from U?; symbol Logic_LevelTranslator:SN74AUP1T34DCK -> bountifulHarvest-rescue:SN74AUP1T34DCK-Logic_LevelTranslator
Changed lines of the file:
@@
 EESchema Schematic File Version 4
-EELAYER 30 0
+LIBS:bountifulHarvest-cache
+EELAYER 26 0
 EELAYER END
 $Descr A4 11693 8268
@@
 F 0 "R5" H 1280 1104 50  0000 R CNN
 F 1 "10k" H 1280 1195 50  0000 R CNN
-F 2 "Resistor_SMD:R_0805_2012Metric_Pad1.15x1.40mm_HandSolder" V 1280 1150 50  0001 C CNN
+F 2 "Resistors_SMD:R_0603_HandSoldering" V 1280 1150 50  0001 C CNN
 F 3 "~" H 1350 1150 50  0001 C CNN
 	1    1350 1150
@@
 F 0 "R3" H 980 1104 50  0000 R CNN
 F 1 "10k" H 980 1195 50  0000 R CNN
-F 2 "Resistor_SMD:R_0805_2012Metric_Pad1.15x1.40mm_HandSolder" V 980 1150 50  0001 C CNN
+F 2 "Resistors_SMD:R_0603_HandSoldering" V 980 1150 50  0001 C CNN
 F 3 "~" H 1050 1150 50  0001 C CNN
 	1    1050 1150
@@
 	10000 3950 8900 3950
 $Comp
-L Logic_LevelTranslator:SN74AUP1T34DCK U?
+L bountifulHarvest-rescue:SN74AUP1T34DCK-Logic_LevelTranslator U201
 U 1 1 63165C49
 P 9350 5900
-F 0 "U?" H 9794 5946 50  0000 L CNN
+F 0 "U201" H 9794 5946 50  0000 L CNN
 F 1 "SN74AUP1T34DCK" H 9794 5855 50  0000 L CNN
 F 2 "Package_TO_SOT_SMD:SOT-353_SC-70-5" H 9350 5200 50  0001 C CNN
@@
 P 9350 6300
 AR Path="/5EE66603/6316E590" Ref="#PWR?"  Part="1"
-AR Path="/5EE7212D/6316E590" Ref="#PWR?"  Part="1"
-F 0 "#PWR?" H 9350 6050 50  0001 C CNN
+AR Path="/5EE7212D/6316E590" Ref="#PWR0280"  Part="1"
+F 0 "#PWR0280" H 9350 6050 50  0001 C CNN
 F 1 "GND" H 9355 6127 50  0000 C CNN
 F 2 "" H 9350 6300 50  0001 C CNN
@@
 	9350 6200 9350 6300
 $Comp
-L power:+3.3V #PWR?
+L power:+3.3V #PWR0281
 U 1 1 631724AF
 P 9250 5400
-F 0 "#PWR?" H 9250 5250 50  0001 C CNN
+F 0 "#PWR0281" H 9250 5250 50  0001 C CNN
 F 1 "+3.3V" H 9265 5573 50  0000 C CNN
 F 2 "" H 9250 5400 50  0001 C CNN
@@
 	9250 5400 9250 5600
 $Comp
-L power:VCC #PWR?
+L power:VCC #PWR0282
 U 1 1 63188529
 P 9500 5400
-F 0 "#PWR?" H 9500 5250 50  0001 C CNN
+F 0 "#PWR0282" H 9500 5250 50  0001 C CNN
 F 1 "VCC" H 9515 5573 50  0000 C CNN
 F 2 "" H 9500 5400 50  0001 C CNN
