File: bountifulHarvest.kicad_pcb (KiCad board)
At the start: 2 copper layers, 114.3 x 114.3 mm, 159 parts, among them J10 CHECK FOOTPRINT, J11 Conn_01x02_Male, J12 CHECK FOOTPRINT, J13 CHECK FOOTPRINT, J14 Conn_01x02_Male, J15 Conn_01x02_Male, J6 CHECK FOOTPRINT, J7 CHECK FOOTPRINT, J8 Conn_01x02_Male, J9 Conn_01x02_Male, Q1 Q_NMOS_GDSD, Q2 Q_NMOS_GDSD, Q3 Q_NMOS_GDSD, Q4 Q_NMOS_GDSD, U1 ATmega2560-16AU, U10 TMC2130-LA, U2 STM32F303CBTx, U3 TPS5431DDA, U4 AMS1117-3.3, U6 TMC2130-LA, U7 TMC2130-LA, U8 TMC2130-LA, U9 TMC2130-LA

Commit message: added peripherals
Parts:
- added R401: .05, Resistors_SMD:R_0603_HandSoldering, F.Cu at (143.0, -93.2)
- added R402: .05, Resistors_SMD:R_0603_HandSoldering, F.Cu at (143.0, -91.8)
- added R403: .05, Resistors_SMD:R_0603_HandSoldering, F.Cu at (146.9, -93.2)
- added R404: 2k, Resistors_SMD:R_0603_HandSoldering, F.Cu at (143.0, -90.3)
- added R405: 2k, Resistors_SMD:R_0603_HandSoldering, F.Cu at (146.9, -91.8)
- added R406: 2k, Resistors_SMD:R_0603_HandSoldering, F.Cu at (143.0, -88.8)
- added R407: 2k, Resistors_SMD:R_0603_HandSoldering, F.Cu at (150.9, -93.2)
- added R408: 2k, Resistors_SMD:R_0603_HandSoldering, F.Cu at (146.9, -90.3)
- added R409: 2k, Resistors_SMD:R_0603_HandSoldering, F.Cu at (150.9, -91.8)
- added R410: 2k, Resistors_SMD:R_0603_HandSoldering, F.Cu at (146.9, -88.8)
- R19: value .02 -> .05
- R23: value 1k -> 2k
Connections:
- net DIAG_0_SPARE renamed /Spare/DIAG_0_SPARE
- R29 pad 1: Net-(R29-Pad1) -> (no net)
- R30 pad 1: Net-(R30-Pad1) -> (no net)
- R31 pad 1: Net-(R31-Pad1) -> (no net)
- R32 pad 2: Net-(R29-Pad1) -> Net-(R32-Pad2)
- R33 pad 2: Net-(R30-Pad1) -> Net-(R33-Pad2)
- R34 pad 2: Net-(R31-Pad1) -> Net-(R34-Pad2)
- R37 pad 1: Net-(R37-Pad1) -> (no net)
- R38 pad 2: Net-(R37-Pad1) -> Net-(R38-Pad2)
- R59 pad 2: /Spare/X2_DIAG -> /Main Processor/X2_4
- TP5 pad 1: /Spare/X2_DIAG -> /Main Processor/X2_4
- U1 pad 21: (no net) -> /Drivers/SCK_SPI
- U1 pad 22: (no net) -> /Drivers/SDI_SPI
- U1 pad 23: (no net) -> /Drivers/SDO_SPI
- U1 pad 63: (no net) -> /Main Processor/X2_0
- U1 pad 64: (no net) -> /Spare/STEP_X2
- U1 pad 65: (no net) -> /Spare/DIR_X2
- U1 pad 66: (no net) -> /Spare/EN_X2
- U1 pad 67: (no net) -> /Main Processor/X2_4
- U10 pad 2: (no net) -> /Main Processor/X2_0
- U10 pad 20: /Spare/X2_DIAG -> /Main Processor/X2_4
- U10 pad 21: /Spare/X2_DIAG -> /Main Processor/X2_4
- U10 pad 22: (no net) -> /Spare/EN_X2
- U10 pad 6: (no net) -> /Spare/STEP_X2
- U10 pad 7: (no net) -> /Spare/DIR_X2

Commit message: added RESET and XTAL to atmega2560
Parts:
- added U5: LM324A, Housings_SOIC:SOIC-14_3.9x8.7mm_Pitch1.27mm, F.Cu at (69.8, 68.6)
- moved U4 196.0 mm to (94.0, 124.5)
- moved U3 192.2 mm to (118.1, 124.5)
- moved J12 187.0 mm to (146.2, 100.9)
- moved J13 187.0 mm to (146.2, 108.0)
- moved U2 172.4 mm to (48.3, 97.3)
- moved R26 166.3 mm to (62.2, 80.0)
- moved C21 166.1 mm to (62.2, 76.2)
- moved J11 162.7 mm to (110.5, 87.6)
- moved J10 162.6 mm to (146.5, 90.2)
- moved R36 161.4 mm to (77.5, 80.0)
- moved J7 159.7 mm to (146.1, 80.0)
- moved C22 158.1 mm to (67.3, 76.2)
- moved C23 152.1 mm to (72.4, 76.2)
- moved R27 149.8 mm to (67.3, 80.0)
- moved R49 149.4 mm to (125.7, 54.6)
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Connections:
- C21 pad 1: /peripherals/P_0_I -> /Main Processor/P_0_I
- C22 pad 1: /peripherals/P_1_I -> /Main Processor/P_1_I
- C23 pad 1: /peripherals/P_2_I -> /Main Processor/P_2_I
- C25 pad 1: /peripherals/P_3_I -> /Main Processor/P_3_I
- R26 pad 1: /peripherals/P_0_I -> /Main Processor/P_0_I
- R27 pad 1: /peripherals/P_1_I -> /Main Processor/P_1_I
- R28 pad 1: /peripherals/P_2_I -> /Main Processor/P_2_I
- R36 pad 1: /peripherals/P_3_I -> /Main Processor/P_3_I
- U1 pad 4: /Drivers/DIR_Y -> /Main Processor/DIR_X
- U1 pad 48: /Drivers/DIR_Y -> /Main Processor/DIR_X
- U1 pad 73: (no net) -> /Main Processor/DIR_X
- U1 pad 74: (no net) -> /Drivers/STEP_X
- U1 pad 75: (no net) -> /Drivers/EN_X
- U1 pad 76: (no net) -> /Drivers/X_0
- U1 pad 94: (no net) -> /Main Processor/P_3_I
- U1 pad 95: (no net) -> /Main Processor/P_2_I
- U1 pad 96: (no net) -> /Main Processor/P_1_I
- U1 pad 97: (no net) -> /Main Processor/P_0_I
- U6 pad 7: /Drivers/DIR_Y -> /Main Processor/DIR_X
- U7 pad 7: /Drivers/DIR_Y -> /Main Processor/DIR_X

Commit message: connected CoP + mP SPI. pushed updated into layout
Parts:
- added C77: .1uF, Resistor_SMD:R_0805_2012Metric_Pad1.15x1.40mm_HandSolder, F.Cu at (92.1, 85.6)
- added C78: .1uF, Resistor_SMD:R_0805_2012Metric_Pad1.15x1.40mm_HandSolder, F.Cu at (92.1, 88.5)
- added C79: .1uF, Resistor_SMD:R_0805_2012Metric_Pad1.15x1.40mm_HandSolder, F.Cu at (96.9, 85.6)
- added C80: 0.1uF, Capacitor_SMD:C_0603_1608Metric_Pad1.05x0.95mm_HandSolder, F.Cu at (106.2, 91.2)
- added C81: 0.1uF, Capacitor_SMD:C_0603_1608Metric_Pad1.05x0.95mm_HandSolder, F.Cu at (110.9, 88.3)
- added C82: 0.1uF, Capacitor_SMD:C_0603_1608Metric_Pad1.05x0.95mm_HandSolder, F.Cu at (59.1, 62.1)
- added C83: DNI, Capacitor_SMD:C_0805_2012Metric_Pad1.15x1.40mm_HandSolder, F.Cu at (30.8, 67.9)
- added C84: DNI, Capacitor_SMD:C_0805_2012Metric_Pad1.15x1.40mm_HandSolder, F.Cu at (35.6, 64.9)
- added C85: DNI, Capacitor_SMD:C_0805_2012Metric_Pad1.15x1.40mm_HandSolder, F.Cu at (47.7, 50.5)
- added C86: DNI, Capacitor_SMD:C_0805_2012Metric_Pad1.15x1.40mm_HandSolder, F.Cu at (30.8, 64.9)
- added C90: DNI, Capacitor_SMD:C_0805_2012Metric_Pad1.15x1.40mm_HandSolder, F.Cu at (35.6, 62.0)
- added C91: DNI, Capacitor_SMD:C_0805_2012Metric_Pad1.15x1.40mm_HandSolder, F.Cu at (30.8, 62.0)
- added C92: DNI, Capacitor_SMD:C_0805_2012Metric_Pad1.15x1.40mm_HandSolder, F.Cu at (54.6, 65.3)
- added C93: DNI, Capacitor_SMD:C_0805_2012Metric_Pad1.15x1.40mm_HandSolder, F.Cu at (40.3, 67.9)
- added R21: 10k, Resistor_SMD:R_0805_2012Metric_Pad1.15x1.40mm_HandSolder, F.Cu at (111.1, 85.6)
- added R22: 10k, Resistor_SMD:R_0805_2012Metric_Pad1.15x1.40mm_HandSolder, F.Cu at (101.6, 94.4)
- added R24: 10k, Resistor_SMD:R_0805_2012Metric_Pad1.15x1.40mm_HandSolder, F.Cu at (96.9, 94.4)
- added R25: 50, Resistor_SMD:R_0805_2012Metric_Pad1.15x1.40mm_HandSolder, F.Cu at (106.4, 85.6)
- added R29: 50, Resistor_SMD:R_0805_2012Metric_Pad1.15x1.40mm_HandSolder, F.Cu at (101.6, 88.5)
- added R3: 10k, Resistor_SMD:R_0805_2012Metric_Pad1.15x1.40mm_HandSolder, F.Cu at (101.6, 91.5)
- added R30: 50, Resistor_SMD:R_0805_2012Metric_Pad1.15x1.40mm_HandSolder, F.Cu at (96.9, 91.5)
- added R31: 50, Resistor_SMD:R_0805_2012Metric_Pad1.15x1.40mm_HandSolder, F.Cu at (92.1, 94.4)
- added R35: 10k, Resistor_SMD:R_0805_2012Metric_Pad1.15x1.40mm_HandSolder, F.Cu at (101.6, 85.6)
- added R37: 10k, Resistor_SMD:R_0805_2012Metric_Pad1.15x1.40mm_HandSolder, F.Cu at (96.9, 88.5)
- added R5: 10k, Resistor_SMD:R_0805_2012Metric_Pad1.15x1.40mm_HandSolder, F.Cu at (106.4, 88.5)
- added R72: 10k, Resistor_SMD:R_0805_2012Metric_Pad1.15x1.40mm_HandSolder, F.Cu at (92.1, 91.5)
- added R75: DNI, Resistor_SMD:R_0805_2012Metric_Pad1.15x1.40mm_HandSolder, F.Cu at (40.3, 62.0)
- added R76: DNI, Resistor_SMD:R_0805_2012Metric_Pad1.15x1.40mm_HandSolder, F.Cu at (47.7, 53.5)
- added R77: DNI, Resistor_SMD:R_0805_2012Metric_Pad1.15x1.40mm_HandSolder, F.Cu at (52.5, 50.5)
- added R78: DNI, Resistor_SMD:R_0805_2012Metric_Pad1.15x1.40mm_HandSolder, F.Cu at (35.6, 67.9)
- added R79: 100, Resistor_SMD:R_0805_2012Metric_Pad1.15x1.40mm_HandSolder, F.Cu at (40.3, 64.9)
- added R80: 100, Resistor_SMD:R_0805_2012Metric_Pad1.15x1.40mm_HandSolder, F.Cu at (47.7, 56.4)
- added R81: 100, Resistor_SMD:R_0805_2012Metric_Pad1.15x1.40mm_HandSolder, F.Cu at (45.1, 62.0)
- added R82: 100, Resistor_SMD:R_0805_2012Metric_Pad1.15x1.40mm_HandSolder, F.Cu at (52.5, 53.5)
- added R83: DNI, Resistor_SMD:R_0805_2012Metric_Pad1.15x1.40mm_HandSolder, F.Cu at (57.2, 50.5)
- added R84: DNI, Resistor_SMD:R_0805_2012Metric_Pad1.15x1.40mm_HandSolder, F.Cu at (59.3, 59.4)
- added R85: DNI, Resistor_SMD:R_0805_2012Metric_Pad1.15x1.40mm_HandSolder, F.Cu at (45.1, 64.9)
- added R86: DNI, Resistor_SMD:R_0805_2012Metric_Pad1.15x1.40mm_HandSolder, F.Cu at (52.5, 56.4)
- added R87: DNI, Resistor_SMD:R_0805_2012Metric_Pad1.15x1.40mm_HandSolder, F.Cu at (49.8, 59.4)
- added R88: DNI, Resistor_SMD:R_0805_2012Metric_Pad1.15x1.40mm_HandSolder, F.Cu at (57.2, 53.5)
- added R89: DNI, Resistor_SMD:R_0805_2012Metric_Pad1.15x1.40mm_HandSolder, F.Cu at (62.0, 50.5)
- added R90: DNI, Resistor_SMD:R_0805_2012Metric_Pad1.15x1.40mm_HandSolder, F.Cu at (49.8, 62.3)
- added R91: 100, Resistor_SMD:R_0805_2012Metric_Pad1.15x1.40mm_HandSolder, F.Cu at (45.1, 67.9)
- added R92: 100, Resistor_SMD:R_0805_2012Metric_Pad1.15x1.40mm_HandSolder, F.Cu at (57.2, 56.4)
- added R93: 100, Resistor_SMD:R_0805_2012Metric_Pad1.15x1.40mm_HandSolder, F.Cu at (54.6, 59.4)
- added R94: 100, Resistor_SMD:R_0805_2012Metric_Pad1.15x1.40mm_HandSolder, F.Cu at (62.0, 53.5)
- added R95: DNI, Resistor_SMD:R_0805_2012Metric_Pad1.15x1.40mm_HandSolder, F.Cu at (49.8, 65.3)
- added R96: DNI, Resistor_SMD:R_0805_2012Metric_Pad1.15x1.40mm_HandSolder, F.Cu at (54.6, 62.3)
- added R97: DNI, Resistor_SMD:R_0805_2012Metric_Pad1.15x1.40mm_HandSolder, F.Cu at (62.0, 56.4)
- added R98: DNI, Resistor_SMD:R_0805_2012Metric_Pad1.15x1.40mm_HandSolder, F.Cu at (49.8, 68.2)
- added U11: AM26LV32xD, Package_SO:SOIC-16_3.9x9.9mm_P1.27mm, F.Cu at (41.1, 54.8)
- added U12: AM26LV32xD, Package_SO:SOIC-16_3.9x9.9mm_P1.27mm, F.Cu at (32.7, 54.8)
- added U3: TPS5430DDA, Package_SO:TI_SO-PowerPAD-8_ThermalVias, F.Cu at (53.6, 111.4)
- moved U1 2.55 mm to (77.5, 95.8)
- moved U2 2.05 mm to (49.3, 95.5)
Connections:
- C38 pad 2: Net-(C38-Pad2) -> +5V
- R11 pad 2: (no net) -> /peripherals/PERIPH_0
- R12 pad 2: (no net) -> /peripherals/PERIPH_1
- R14 pad 2: (no net) -> /peripherals/PERIPH_2
- R16 pad 2: (no net) -> /peripherals/PERIPH_3
- R404 pad 2: (no net) -> /peripherals/P_1_SENSE
- R405 pad 2: (no net) -> /peripherals/P_2_SENSE
- R409 pad 2: (no net) -> /peripherals/P_3_SENSE
- U1 pad 1: (no net) -> Net-(U1-Pad1)
- U1 pad 10: Net-(U1-Pad10) -> +5V
- U1 pad 100: (no net) -> Net-(C96-Pad1)
- U1 pad 11: Net-(U1-Pad11) -> GND
- U1 pad 12: /Drivers/Z_0 -> Net-(U1-Pad12)
- U1 pad 13: /Drivers/Z_1 -> Net-(U1-Pad13)
- U1 pad 14: /Drivers/Z_2 -> Net-(U1-Pad14)
- U1 pad 15: /Drivers/Z_3 -> /peripherals/PERIPH_0
- U1 pad 16: /Drivers/Z_4 -> /peripherals/PERIPH_1
- U1 pad 17: (no net) -> /peripherals/PERIPH_2
- U1 pad 18: (no net) -> /peripherals/PERIPH_3
- U1 pad 19: (no net) -> /Main Processor/~CS~_SPI
- U1 pad 2: /Drivers/Y_0 -> Net-(U1-Pad2)
- U1 pad 20: (no net) -> /SCK
- U1 pad 21: /Drivers/SCK_SPI -> /MISO
- U1 pad 22: /Drivers/SDI_SPI -> /MOSI
- U1 pad 23: /Drivers/SDO_SPI -> Net-(U1-Pad23)
- U1 pad 24: (no net) -> Net-(U1-Pad24)
- U1 pad 25: (no net) -> Net-(U1-Pad25)
- U1 pad 26: (no net) -> Net-(U1-Pad26)
- U1 pad 27: (no net) -> Net-(U1-Pad27)
- U1 pad 28: (no net) -> Net-(U1-Pad28)
- U1 pad 29: (no net) -> Net-(U1-Pad29)
- U1 pad 30: (no net) -> /Main Processor/~RESET
- U1 pad 31: Net-(U1-Pad10) -> +5V
- U1 pad 32: Net-(U1-Pad11) -> GND
- U1 pad 33: (no net) -> Net-(C98-Pad1)
- U1 pad 34: (no net) -> Net-(C97-Pad1)
- U1 pad 35: (no net) -> /Main Processor/COP_RESET
- U1 pad 36: (no net) -> /Main Processor/PL1
- U1 pad 37: (no net) -> /Main Processor/DIA_X2
- U1 pad 38: (no net) -> /Main Processor/DIA_X1
- U1 pad 39: (no net) -> /Main Processor/DIA_Y
- U1 pad 40: (no net) -> /Main Processor/DIA_Z
- U1 pad 41: (no net) -> /Main Processor/DIA_AUX
- U1 pad 42: (no net) -> /Main Processor/PL2
- U1 pad 43: (no net) -> /Main Processor/SCL
- U1 pad 44: (no net) -> /Main Processor/SDA
- U1 pad 45: (no net) -> Net-(U1-Pad45)
- U1 pad 46: /Drivers/X_0 -> Net-(U1-Pad46)
- U1 pad 47: /Drivers/STEP_X -> Net-(U1-Pad47)
- U1 pad 48: /Main Processor/DIR_X -> Net-(U1-Pad48)
- U1 pad 49: /Drivers/EN_X -> Net-(U1-Pad49)
- U1 pad 50: /Drivers/X_4 -> Net-(U1-Pad50)
- U1 pad 51: (no net) -> Net-(U1-Pad51)
- U1 pad 52: (no net) -> Net-(U1-Pad52)
- U1 pad 53: (no net) -> Net-(U1-Pad53)
- U1 pad 54: (no net) -> Net-(U1-Pad54)
- U1 pad 55: (no net) -> Net-(U1-Pad55)
- U1 pad 56: (no net) -> Net-(U1-Pad56)
- U1 pad 57: (no net) -> Net-(U1-Pad57)
- U1 pad 58: (no net) -> Net-(U1-Pad58)
- U1 pad 59: (no net) -> Net-(U1-Pad59)
- U1 pad 60: (no net) -> Net-(U1-Pad60)
- U1 pad 61: Net-(U1-Pad10) -> +5V
- U1 pad 62: Net-(U1-Pad11) -> GND
- U1 pad 63: /Main Processor/X2_0 -> /Main Processor/X2_STEP
- U1 pad 64: /Spare/STEP_X2 -> /Main Processor/X2_EN
- U1 pad 65: /Spare/DIR_X2 -> Net-(U1-Pad65)
- U1 pad 66: /Spare/EN_X2 -> Net-(U1-Pad66)
- U1 pad 67: /Main Processor/X2_4 -> Net-(U1-Pad67)
- U1 pad 68: (no net) -> Net-(U1-Pad68)
- U1 pad 69: (no net) -> Net-(U1-Pad69)
- U1 pad 7: (no net) -> Net-(U1-Pad7)
- U1 pad 70: (no net) -> Net-(U1-Pad70)
- U1 pad 71: (no net) -> /Main Processor/~CS_X2
- U1 pad 72: (no net) -> /Main Processor/~CS_Y
- U1 pad 73: /Main Processor/DIR_X -> /Main Processor/X1_DIR
- U1 pad 74: /Drivers/STEP_X -> /Main Processor/X1_STEP
- U1 pad 75: /Drivers/EN_X -> /Main Processor/X1_EN
- U1 pad 76: /Drivers/X_0 -> /Main Processor/~CS_X1
- U1 pad 77: (no net) -> /Main Processor/~CS_Z
- U1 pad 78: (no net) -> /Coprocessor/~CS
- U1 pad 79: (no net) -> Net-(U1-Pad79)
- U1 pad 8: (no net) -> Net-(U1-Pad8)
- U1 pad 80: Net-(U1-Pad10) -> +5V
- U1 pad 81: Net-(U1-Pad11) -> GND
- U1 pad 82: (no net) -> /Main Processor/X_MIN
- U1 pad 83: (no net) -> /Main Processor/X_MAX
- U1 pad 84: (no net) -> /Main Processor/Y_MIN
- U1 pad 85: (no net) -> /Main Processor/Y_MAX
- U1 pad 86: (no net) -> /Main Processor/Z_MIN
- U1 pad 87: (no net) -> /Main Processor/Z_MAX
- U1 pad 88: (no net) -> /Main Processor/PK1
- U1 pad 89: (no net) -> /Main Processor/PK0
- U1 pad 9: (no net) -> Net-(U1-Pad9)
- U1 pad 90: (no net) -> Net-(U1-Pad90)
- U1 pad 91: (no net) -> Net-(U1-Pad91)
- U1 pad 92: (no net) -> Net-(U1-Pad92)
- U1 pad 93: (no net) -> Net-(U1-Pad93)
- U1 pad 94: /Main Processor/P_3_I -> Net-(U1-Pad94)
- U1 pad 95: /Main Processor/P_2_I -> Net-(U1-Pad95)
- U1 pad 98: (no net) -> Net-(U1-Pad98)
- U1 pad 99: Net-(U1-Pad11) -> GND
- U10 pad 10: (no net) -> Net-(U10-Pad10)
- U10 pad 17: (no net) -> Net-(U10-Pad17)
- U10 pad 19: (no net) -> Net-(U10-Pad19)
- U10 pad 3: /Drivers/SCK_SPI -> /SCK
- U10 pad 30: (no net) -> +5V
- U10 pad 4: /Drivers/SDI_SPI -> /MISO
- U10 pad 5: /Drivers/SDO_SPI -> /MOSI
- U10 pad 9: (no net) -> Net-(U10-Pad9)
- U2 pad 1: (no net) -> +3V3
- U2 pad 10: (no net) -> /Coprocessor/Z_A_ENC
- U2 pad 11: (no net) -> /Coprocessor/Z_A_ENC
- U2 pad 12: (no net) -> Net-(U2-Pad12)
- U2 pad 13: (no net) -> Net-(U2-Pad13)
- U2 pad 14: (no net) -> Net-(R25-Pad2)
- U2 pad 15: (no net) -> Net-(R29-Pad2)
- U2 pad 16: (no net) -> Net-(R30-Pad2)
- U2 pad 17: (no net) -> Net-(R31-Pad2)
- U2 pad 18: (no net) -> Net-(U2-Pad18)
- U2 pad 19: (no net) -> Net-(U2-Pad19)
- U2 pad 2: (no net) -> Net-(U2-Pad2)
- U2 pad 20: (no net) -> Net-(U2-Pad20)
- U2 pad 21: (no net) -> Net-(U2-Pad21)
- U2 pad 22: (no net) -> Net-(U2-Pad22)
- U2 pad 23: (no net) -> GND
- U2 pad 24: (no net) -> +3V3
- U2 pad 25: (no net) -> Net-(U2-Pad25)
- U2 pad 26: (no net) -> Net-(U2-Pad26)
- U2 pad 27: (no net) -> Net-(U2-Pad27)
- U2 pad 28: (no net) -> Net-(U2-Pad28)
- U2 pad 29: (no net) -> /Coprocessor/X1_A_ENC
- U2 pad 3: (no net) -> Net-(U2-Pad3)
- U2 pad 30: (no net) -> /Coprocessor/X1_B_ENC
- U2 pad 31: (no net) -> Net-(U2-Pad31)
- U2 pad 32: (no net) -> /Coprocessor/X0_A_ENC
- U2 pad 33: (no net) -> /Coprocessor/X0_B_ENC
- U2 pad 34: (no net) -> /Coprocessor/SWDIO
- U2 pad 35: (no net) -> GND
- U2 pad 36: (no net) -> +3V3
- U2 pad 37: (no net) -> /Coprocessor/SWDCLK
- U2 pad 38: (no net) -> Net-(U2-Pad38)
- U2 pad 39: (no net) -> Net-(U2-Pad39)
- U2 pad 4: (no net) -> Net-(U2-Pad4)
- U2 pad 40: (no net) -> /Coprocessor/Y_A_ENC
- U2 pad 41: (no net) -> /Coprocessor/Y_B_ENC
- U2 pad 42: (no net) -> Net-(U2-Pad42)
- U2 pad 43: (no net) -> Net-(U2-Pad43)
- U2 pad 44: (no net) -> Net-(R22-Pad1)
- U2 pad 45: (no net) -> Net-(U2-Pad45)
- U2 pad 46: (no net) -> Net-(U2-Pad46)
- U2 pad 47: (no net) -> GND
- U2 pad 48: (no net) -> +3V3
- U2 pad 5: (no net) -> Net-(R24-Pad1)
- U2 pad 6: (no net) -> Net-(U2-Pad6)
- U2 pad 7: (no net) -> /Coprocessor/~COP_RESET
- U2 pad 8: (no net) -> GND
- U2 pad 9: (no net) -> Net-(C80-Pad1)
- U6 pad 10: (no net) -> Net-(U6-Pad10)
- U6 pad 17: (no net) -> Net-(U6-Pad17)
- U6 pad 19: (no net) -> Net-(U6-Pad19)
- U6 pad 3: /Drivers/SCK_SPI -> /SCK
- U6 pad 30: (no net) -> +5V
- U6 pad 4: /Drivers/SDI_SPI -> /MISO
- U6 pad 5: /Drivers/SDO_SPI -> /MOSI
- U6 pad 9: (no net) -> Net-(U6-Pad9)
- U7 pad 10: (no net) -> Net-(U7-Pad10)
- U7 pad 17: (no net) -> Net-(U7-Pad17)
- U7 pad 19: (no net) -> Net-(U7-Pad19)
- U7 pad 3: /Drivers/SCK_SPI -> /SCK
- U7 pad 30: (no net) -> +5V
- U7 pad 4: /Drivers/SDI_SPI -> /MISO
- U7 pad 5: /Drivers/SDO_SPI -> /MOSI
- U7 pad 9: (no net) -> Net-(U7-Pad9)
- U8 pad 10: (no net) -> Net-(U8-Pad10)
- U8 pad 17: (no net) -> Net-(U8-Pad17)
- U8 pad 19: (no net) -> Net-(U8-Pad19)
- U8 pad 25: Net-(C38-Pad2) -> +5V
- U8 pad 3: /Drivers/SCK_SPI -> /SCK
- U8 pad 30: (no net) -> +5V
- U8 pad 4: /Drivers/SDI_SPI -> /MISO
- U8 pad 5: /Drivers/SDO_SPI -> /MOSI
- U8 pad 9: (no net) -> Net-(U8-Pad9)
- U9 pad 10: (no net) -> Net-(U9-Pad10)
- U9 pad 17: (no net) -> Net-(U9-Pad17)
- U9 pad 19: (no net) -> Net-(U9-Pad19)
- U9 pad 2: (no net) -> /Spare/SPARE_0
- U9 pad 22: (no net) -> /Spare/EN_SPARE
- U9 pad 3: /Drivers/SCK_SPI -> /SCK
- U9 pad 30: (no net) -> +5V
- U9 pad 4: /Drivers/SDI_SPI -> /MISO
- U9 pad 5: /Drivers/SDO_SPI -> /MOSI
- U9 pad 6: (no net) -> /Spare/SPARE_1
- U9 pad 7: (no net) -> /Spare/DIR_SPARE
- U9 pad 9: (no net) -> Net-(U9-Pad9)

Commit message: added footprints for most of the c,r, and tp's. need new buck
Parts:
- removed the U3 at (53.6, 111.4)
- added C87: 1uF, Capacitors_SMD:C_0603_HandSoldering, F.Cu at (214.1, -141.5)
- added C88: 1uF, Capacitors_SMD:C_0603_HandSoldering, F.Cu at (210.4, -140.1)
- added C89: 0.1uF, Capacitors_SMD:C_0603_HandSoldering, F.Cu at (214.1, -142.8)
- added C901: .1uF, Capacitors_SMD:C_0603_HandSoldering, F.Cu at (201.1, -142.8)
- added C902: 1uF, Capacitors_SMD:C_0603_HandSoldering, F.Cu at (203.6, -138.8)
- added C903: 22uF, Capacitors_SMD:C_0603_HandSoldering, F.Cu at (200.0, -138.8)
- added C904: 22uF, Capacitors_SMD:C_0603_HandSoldering, F.Cu at (201.1, -140.1)
- added C905: 10uF, Capacitors_SMD:C_0603_HandSoldering, F.Cu at (201.1, -141.5)
- added C906: 1uF, Capacitors_SMD:C_0603_HandSoldering, F.Cu at (196.3, -139.1)
- added C94: 1uF, Capacitors_SMD:C_0603_HandSoldering, F.Cu at (210.4, -142.8)
- added C95: 1uF, Capacitors_SMD:C_0603_HandSoldering, F.Cu at (210.4, -141.5)
- added C97: 20pF, Capacitors_SMD:C_0603_HandSoldering, F.Cu at (185.8, -137.2)
- added C98: 20pF, Capacitors_SMD:C_0603_HandSoldering, F.Cu at (189.2, -139.9)
- added D15: LED, LEDs:LED_0805_HandSoldering, F.Cu at (177.6, -128.6)
- added D16: LED, LEDs:LED_0805_HandSoldering, F.Cu at (177.6, -130.4)
- added D901: LED, LEDs:LED_0805_HandSoldering, F.Cu at (196.9, -140.7)
- added D902: LED, LEDs:LED_0805_HandSoldering, F.Cu at (196.9, -142.6)
- added R1: 10K, Resistors_SMD:R_0603_HandSoldering, F.Cu at (185.2, -135.6)
- added R100: 1M, Resistors_SMD:R_0805_HandSoldering, F.Cu at (177.6, -136.9)
- added R101: 10K, Resistors_SMD:R_0603_HandSoldering, F.Cu at (181.2, -135.2)
- added R102: 10K, Resistors_SMD:R_0603_HandSoldering, F.Cu at (189.4, -141.3)
- added R103: 10K, Resistors_SMD:R_0603_HandSoldering, F.Cu at (177.2, -135.2)
- added R106: 10k, Resistors_SMD:R_0603_HandSoldering, F.Cu at (182.0, -137.1)
- added R2: 10K, Resistors_SMD:R_0603_HandSoldering, F.Cu at (189.4, -142.8)
- added R39: 10, Resistors_SMD:R_0603_HandSoldering, F.Cu at (194.4, -130.6)
- added R4: 10k, Resistors_SMD:R_0603_HandSoldering, F.Cu at (186.3, -129.1)
- added R40: 10, Resistors_SMD:R_0603_HandSoldering, F.Cu at (194.4, -129.1)
- added R51: 10, Resistors_SMD:R_0603_HandSoldering, F.Cu at (198.4, -130.6)
- added R57: 10, Resistors_SMD:R_0603_HandSoldering, F.Cu at (205.6, -133.5)
- added R58: 10, Resistors_SMD:R_0603_HandSoldering, F.Cu at (205.6, -132.1)
- added R6: 3.34k, Resistors_SMD:R_0603_HandSoldering, F.Cu at (181.6, -125.1)
- added R73: R, Resistors_SMD:R_0603_HandSoldering, F.Cu at (186.3, -130.6)
- added R74: R, Resistors_SMD:R_0603_HandSoldering, F.Cu at (177.2, -124.2)
- added TP1: TestPoint, Measurement_Points:Test_Point_Keystone_5015_Micro-Minature, F.Cu at (182.2, -130.0)
- added TP301: TestPoint, Measurement_Points:Test_Point_Keystone_5015_Micro-Minature, F.Cu at (182.2, -127.2)
- added TP8: TestPoint, Measurement_Points:Test_Point_Keystone_5015_Micro-Minature, F.Cu at (177.4, -126.3)
- added Y1: 16MHz, Crystals:Crystal_HC49-4H_Vertical, F.Cu at (178.9, -140.7)
- R20: value .02 -> R
- R21, R22: value .02 -> 10k
- R24, R35, R37: value 1k -> 10k
- R25, R29, R30, R31: value 1k -> 50
- U3: value TPS5431DDA -> TPS5430DDA
- moved C65 276.6 mm to (-22.4, 60.2)
- moved C66 276.6 mm to (-29.7, 62.8)
- moved C67 276.6 mm to (-34.2, 62.3)
- moved C68 276.6 mm to (-29.7, 64.6)
- moved C72 276.6 mm to (-23.3, 56.6)
- moved D13 276.6 mm to (-25.5, 65.8)
- moved J15 276.6 mm to (-27.4, 55.7)
- moved R59 276.6 mm to (-95.2, 60.1)
- moved R60 276.6 mm to (-90.4, 60.1)
- moved R61 276.6 mm to (-80.6, 51.8)
- moved R62 276.6 mm to (-25.4, 62.6)
- moved R63 276.6 mm to (-45.7, 61.3)
- moved R65 276.6 mm to (-85.7, 60.1)
- moved R70 276.6 mm to (-80.6, 54.7)
- moved TP7 276.6 mm to (-18.4, 62.7)
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Connections:
- R20 pad 1: Net-(Q2-Pad3) -> +3V3
- R20 pad 2: GND -> Net-(C80-Pad1)
- R21 pad 1: Net-(Q3-Pad3) -> GND
- R21 pad 2: GND -> /Coprocessor/SWDCLK
- R22 pad 1: Net-(Q4-Pad3) -> Net-(R22-Pad1)
- R24 pad 1: Net-(C19-Pad1) -> Net-(R24-Pad1)
- R24 pad 2: (no net) -> GND
- R25 pad 1: Net-(C20-Pad1) -> /Coprocessor/~CS
- R25 pad 2: (no net) -> Net-(R25-Pad2)
- R29 pad 1: (no net) -> /MOSI
- R29 pad 2: GND -> Net-(R29-Pad2)
- R30 pad 2: GND -> Net-(R30-Pad2)
- R31 pad 1: (no net) -> /SCK
- R31 pad 2: GND -> Net-(R31-Pad2)
- R35 pad 1: Net-(C24-Pad1) -> GND
- R35 pad 2: (no net) -> /Coprocessor/~CS
- R37 pad 1: (no net) -> GND
- R37 pad 2: GND -> /MOSI
- R404 pad 2: /peripherals/P_1_SENSE -> (no net)
- R405 pad 2: /peripherals/P_2_SENSE -> (no net)
- R409 pad 2: /peripherals/P_3_SENSE -> (no net)
- R5 pad 1: Net-(J16-Pad1) -> (no net)
- U1 pad 1: Net-(U1-Pad1) -> (no net)
- U1 pad 100: Net-(C96-Pad1) -> (no net)
- U1 pad 12: Net-(U1-Pad12) -> (no net)
- U1 pad 13: Net-(U1-Pad13) -> (no net)
- U1 pad 14: Net-(U1-Pad14) -> (no net)
- U1 pad 2: Net-(U1-Pad2) -> (no net)
- U1 pad 23: Net-(U1-Pad23) -> (no net)
- U1 pad 24: Net-(U1-Pad24) -> (no net)
- U1 pad 25: Net-(U1-Pad25) -> (no net)
- U1 pad 26: Net-(U1-Pad26) -> (no net)
- U1 pad 27: Net-(U1-Pad27) -> (no net)
- U1 pad 28: Net-(U1-Pad28) -> (no net)
- U1 pad 29: Net-(U1-Pad29) -> (no net)
- U1 pad 36: /Main Processor/PL1 -> (no net)
- U1 pad 37: /Main Processor/DIA_X2 -> (no net)
- U1 pad 38: /Main Processor/DIA_X1 -> (no net)
- U1 pad 39: /Main Processor/DIA_Y -> (no net)
- U1 pad 40: /Main Processor/DIA_Z -> (no net)
- U1 pad 41: /Main Processor/DIA_AUX -> (no net)
- U1 pad 42: /Main Processor/PL2 -> (no net)
- U1 pad 43: /Main Processor/SCL -> (no net)
- U1 pad 44: /Main Processor/SDA -> (no net)
- U1 pad 45: Net-(U1-Pad45) -> (no net)
- U1 pad 46: Net-(U1-Pad46) -> (no net)
- U1 pad 47: Net-(U1-Pad47) -> (no net)
- U1 pad 48: Net-(U1-Pad48) -> (no net)
- U1 pad 49: Net-(U1-Pad49) -> (no net)
- U1 pad 50: Net-(U1-Pad50) -> (no net)
- U1 pad 51: Net-(U1-Pad51) -> (no net)
- U1 pad 52: Net-(U1-Pad52) -> (no net)
- U1 pad 53: Net-(U1-Pad53) -> (no net)
- U1 pad 54: Net-(U1-Pad54) -> (no net)
- U1 pad 55: Net-(U1-Pad55) -> (no net)
- U1 pad 56: Net-(U1-Pad56) -> (no net)
- U1 pad 57: Net-(U1-Pad57) -> (no net)
- U1 pad 58: Net-(U1-Pad58) -> (no net)
- U1 pad 59: Net-(U1-Pad59) -> (no net)
- U1 pad 60: Net-(U1-Pad60) -> (no net)
- U1 pad 63: /Main Processor/X2_STEP -> (no net)
- U1 pad 64: /Main Processor/X2_EN -> (no net)
- U1 pad 65: Net-(U1-Pad65) -> (no net)
- U1 pad 66: Net-(U1-Pad66) -> (no net)
- U1 pad 67: Net-(U1-Pad67) -> (no net)
- U1 pad 68: Net-(U1-Pad68) -> (no net)
- U1 pad 69: Net-(U1-Pad69) -> (no net)
- U1 pad 7: Net-(U1-Pad7) -> (no net)
- U1 pad 70: Net-(U1-Pad70) -> (no net)
- U1 pad 71: /Main Processor/~CS_X2 -> (no net)
- U1 pad 72: /Main Processor/~CS_Y -> (no net)
- U1 pad 73: /Main Processor/X1_DIR -> (no net)
- U1 pad 74: /Main Processor/X1_STEP -> (no net)
- U1 pad 75: /Main Processor/X1_EN -> (no net)
- U1 pad 76: /Main Processor/~CS_X1 -> (no net)
- U1 pad 77: /Main Processor/~CS_Z -> (no net)
- U1 pad 79: Net-(U1-Pad79) -> (no net)
- U1 pad 8: Net-(U1-Pad8) -> (no net)
- U1 pad 82: /Main Processor/X_MIN -> (no net)
- U1 pad 83: /Main Processor/X_MAX -> (no net)
- U1 pad 84: /Main Processor/Y_MIN -> (no net)
- U1 pad 85: /Main Processor/Y_MAX -> (no net)
- U1 pad 86: /Main Processor/Z_MIN -> (no net)
- U1 pad 87: /Main Processor/Z_MAX -> (no net)
- U1 pad 88: /Main Processor/PK1 -> (no net)
- U1 pad 89: /Main Processor/PK0 -> (no net)
- U1 pad 9: Net-(U1-Pad9) -> (no net)
- U1 pad 90: Net-(U1-Pad90) -> (no net)
- U1 pad 91: Net-(U1-Pad91) -> (no net)
- U1 pad 92: Net-(U1-Pad92) -> (no net)
- U1 pad 93: Net-(U1-Pad93) -> (no net)
- U1 pad 94: Net-(U1-Pad94) -> (no net)
- U1 pad 95: Net-(U1-Pad95) -> (no net)
- U1 pad 98: Net-(U1-Pad98) -> (no net)
- U10 pad 10: Net-(U10-Pad10) -> (no net)
- U10 pad 17: Net-(U10-Pad17) -> (no net)
- U10 pad 19: Net-(U10-Pad19) -> (no net)
- U10 pad 2: /Main Processor/X2_0 -> (no net)
- U10 pad 22: /Spare/EN_X2 -> (no net)
- U10 pad 6: /Spare/STEP_X2 -> (no net)
- U10 pad 7: /Spare/DIR_X2 -> (no net)
- U10 pad 9: Net-(U10-Pad9) -> (no net)
- U11 pad 4: Net-(U11-Pad4) -> (no net)
- U12 pad 4: Net-(U12-Pad4) -> (no net)
- U2 pad 12: Net-(U2-Pad12) -> (no net)
- U2 pad 13: Net-(U2-Pad13) -> (no net)
- U2 pad 18: Net-(U2-Pad18) -> (no net)
- U2 pad 19: Net-(U2-Pad19) -> (no net)
- U2 pad 2: Net-(U2-Pad2) -> (no net)
- U2 pad 20: Net-(U2-Pad20) -> (no net)
- U2 pad 21: Net-(U2-Pad21) -> (no net)
- U2 pad 22: Net-(U2-Pad22) -> (no net)
- U2 pad 25: Net-(U2-Pad25) -> (no net)
- U2 pad 26: Net-(U2-Pad26) -> (no net)
- U2 pad 27: Net-(U2-Pad27) -> (no net)
- U2 pad 28: Net-(U2-Pad28) -> (no net)
- U2 pad 3: Net-(U2-Pad3) -> (no net)
- U2 pad 31: Net-(U2-Pad31) -> (no net)
- U2 pad 38: Net-(U2-Pad38) -> (no net)
- U2 pad 39: Net-(U2-Pad39) -> (no net)
- U2 pad 4: Net-(U2-Pad4) -> (no net)
- U2 pad 42: Net-(U2-Pad42) -> (no net)
- U2 pad 43: Net-(U2-Pad43) -> (no net)
- U2 pad 45: Net-(U2-Pad45) -> (no net)
- U2 pad 46: Net-(U2-Pad46) -> (no net)
- U2 pad 6: Net-(U2-Pad6) -> (no net)
- U3 pad 4: (no net) -> Net-(R4-Pad2)
- U3 pad 5: (no net) -> Net-(TP8-Pad1)
- U6 pad 10: Net-(U6-Pad10) -> (no net)
- U6 pad 17: Net-(U6-Pad17) -> (no net)
- U6 pad 19: Net-(U6-Pad19) -> (no net)
- U6 pad 2: /Drivers/Y_0 -> (no net)
- U6 pad 9: Net-(U6-Pad9) -> (no net)
- U7 pad 10: Net-(U7-Pad10) -> (no net)
- U7 pad 17: Net-(U7-Pad17) -> (no net)
- U7 pad 19: Net-(U7-Pad19) -> (no net)
- U7 pad 2: /Drivers/X_0 -> (no net)
- U7 pad 22: /Drivers/EN_X -> (no net)
- U7 pad 6: /Drivers/STEP_X -> (no net)
- U7 pad 9: Net-(U7-Pad9) -> (no net)
- U8 pad 10: Net-(U8-Pad10) -> (no net)
- U8 pad 17: Net-(U8-Pad17) -> (no net)
- U8 pad 19: Net-(U8-Pad19) -> (no net)
- U8 pad 2: /Drivers/Z_0 -> (no net)
- U8 pad 22: /Drivers/Z_3 -> (no net)
- U8 pad 6: /Drivers/Z_1 -> (no net)
- U8 pad 7: /Drivers/Z_2 -> (no net)
- U8 pad 9: Net-(U8-Pad9) -> (no net)
- U9 pad 10: Net-(U9-Pad10) -> (no net)
- U9 pad 17: Net-(U9-Pad17) -> (no net)
- U9 pad 19: Net-(U9-Pad19) -> (no net)
- U9 pad 2: /Spare/SPARE_0 -> (no net)
- U9 pad 22: /Spare/EN_SPARE -> (no net)
- U9 pad 6: /Spare/SPARE_1 -> (no net)
- U9 pad 7: /Spare/DIR_SPARE -> (no net)
- U9 pad 9: Net-(U9-Pad9) -> (no net)
Other:
- copper layers 2 -> 4
